File: electrical/control/control.kicad_pcb (KiCad board)
At the start: 2 copper layers, 30 x 45 mm, 46 parts, among them J1 USB4105-GF-A, J2 UART, J3 SWD, J4 TC2030-NL, J5 QWIIC, SW1 SYS, U1 USBLC6-2P6, U2 LP5912-3.3DRV, U3 W25Q16JVUXIQ, U4 RP2040, U5 ABPMRRV060MG2A3, Y1 ABM8-272-T3

Commit message: Replace I2C connector
Parts:
- added C19: 100n, Capacitor_SMD:C_0402_1005Metric, F.Cu at (138.0, 107.2)
- added R6: 2k2, Resistor_SMD:R_0402_1005Metric, F.Cu at (136.2, 106.6)
- added R7: 2k2, Resistor_SMD:R_0402_1005Metric, F.Cu at (139.8, 106.6)
- J5: value QWIIC -> I2C; footprint Connector_JST:JST_SH_SM04B-SRSS-TB_1x04-1MP_P1.00mm_Horizontal -> Connector_Molex:Molex_PicoBlade_53261-0471_1x04-1MP_P1.25mm_Horizontal
- moved J5 14.0 mm to (138.0, 111.4)
- moved C18 12.0 mm to (158.0, 109.9)
- moved U5 12.0 mm to (151.0, 110.4)
- moved J4 0.40 mm to (155.6, 103.6)
- renumbered LP1 to H2, R9 to R10, R8 to R11, R10 to R12, R11 to R13, R6 to R4, R7 to R5, R4 to R8, R5 to R9
Connections:
- J5 pad 1: GND -> I2C_SDA
- J5 pad 3: I2C_SDA -> GND
Routing:
- net +3.3V: track 102.6 -> 117.5 mm, vias 8 -> 10
- net I2C_SDA: track 44.8 -> 31.0 mm
- net PRESSURE_INT: track 31.5 -> 41.5 mm, vias 0 -> 2
- net I2C_SCL: track 36.5 -> 29.1 mm
- net GND: track 53.4 -> 55.2 mm
Other:
- board text removed: "QWIIC"
