File: electrical/control/control.kicad_sch (KiCad schematic)
At the start: 42 parts, among them J1 USB4105-GF-A, J2 SWD, J3 TC2030-NL, J4 UART, J5 QWIIC, SW1 228EMSARGFR, U1 USBLC6-2P6, U2 LP5912-3.3DRV, U3 W25Q16JVUXIQ, U4 RP2040, U5 ABPMRRV060MG2A3, Y1 ABM8-272-T3

Commit message: Position mechanical components
Parts:
- renumbered J4 to J2, J2 to J3, J3 to J4
Other:
- moved on the sheet: J2, J3
Changed lines of the file:
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@@
 	)
 	(no_connect
-		(at 54.61 203.2)
+		(at 54.61 218.44)
 	)
 	(no_connect
@@
 	)
 	(no_connect
-		(at 54.61 218.44)
+		(at 54.61 203.2)
 	)
 	(no_connect
@@
 	(wire
 		(pts
-			(xy 62.23 195.58) (xy 62.23 200.66)
+			(xy 62.23 210.82) (xy 62.23 215.9)
 		)
 		(stroke
@@
 	(wire
 		(pts
-			(xy 59.69 195.58) (xy 62.23 195.58)
+			(xy 59.69 210.82) (xy 62.23 210.82)
 		)
 		(stroke
@@
 	(wire
 		(pts
-			(xy 62.23 210.82) (xy 62.23 215.9)
+			(xy 62.23 195.58) (xy 62.23 200.66)
 		)
 		(stroke
@@
 	(wire
 		(pts
-			(xy 59.69 193.04) (xy 64.77 193.04)
+			(xy 59.69 208.28) (xy 64.77 208.28)
 		)
 		(stroke
@@
 	(wire
 		(pts
-			(xy 59.69 210.82) (xy 62.23 210.82)
+			(xy 59.69 195.58) (xy 62.23 195.58)
 		)
 		(stroke
@@
 	(wire
 		(pts
-			(xy 59.69 208.28) (xy 64.77 208.28)
+			(xy 59.69 193.04) (xy 64.77 193.04)
 		)
 		(stroke
@@
 	(wire
 		(pts
-			(xy 59.69 198.12) (xy 64.77 198.12)
+			(xy 59.69 213.36) (xy 64.77 213.36)
 		)
 		(stroke
@@
 	(wire
 		(pts
-			(xy 59.69 213.36) (xy 64.77 213.36)
+			(xy 59.69 198.12) (xy 64.77 198.12)
 		)
 		(stroke
@@
 	(global_label "UART_TX"
 		(shape input)
-		(at 64.77 213.36 0)
+		(at 64.77 198.12 0)
 		(fields_autoplaced yes)
 		(effects
@@
 		)
 		(property "Intersheetrefs" "${INTERSHEET_REFS}"
-			(at 75.5566 213.36 0)
+			(at 75.5566 198.12 0)
 			(effects
 				(font
@@
 	(global_label "UART_RX"
 		(shape output)
-		(at 64.77 208.28 0)
+		(at 64.77 193.04 0)
 		(fields_autoplaced yes)
 		(effects
@@
 		)
 		(property "Intersheetrefs" "${INTERSHEET_REFS}"
-			(at 75.859 208.28 0)
+			(at 75.859 193.04 0)
 			(effects
 				(font
@@
 	(global_label "SWCLK"
 		(shape output)
-		(at 64.77 193.04 0)
+		(at 64.77 208.28 0)
 		(fields_autoplaced yes)
 		(effects
@@
 		)
 		(property "Intersheetrefs" "${INTERSHEET_REFS}"
-			(at 73.9842 193.04 0)
+			(at 73.9842 208.28 0)
 			(effects
 				(font
@@
 	(global_label "SWDIO"
 		(shape bidirectional)
-		(at 64.77 198.12 0)
+		(at 64.77 213.36 0)
 		(fields_autoplaced yes)
 		(effects
@@
 		)
 		(property "Intersheetrefs" "${INTERSHEET_REFS}"
-			(at 74.7327 198.12 0)
+			(at 74.7327 213.36 0)
 			(effects
 				(font
@@
 	(symbol
 		(lib_id "Connector_Generic_MountingPin:Conn_01x03_MountingPin")
-		(at 54.61 210.82 0)
+		(at 54.61 195.58 0)
 		(mirror y)
 		(unit 1)
@@
 		(on_board yes)
 		(dnp no)
-		(property "Reference" "J4"
-			(at 52.07 209.9055 0)
+		(property "Reference" "J2"
+			(at 52.07 194.6655 0)
 			(effects
 				(font
@@
 		)
 		(property "Value" "UART"
-			(at 52.07 212.4455 0)
+			(at 52.07 197.2055 0)
 			(effects
 				(font
@@
 		)
 		(property "Footprint" "Connector_JST:JST_SH_SM03B-SRSS-TB_1x03-1MP_P1.00mm_Horizontal"
-			(at 54.61 210.82 0)
+			(at 54.61 195.58 0)
 			(effects
 				(font
@@
 		)
 		(property "Datasheet" "~"
-			(at 54.61 210.82 0)
+			(at 54.61 195.58 0)
 			(effects
 				(font
@@
 		)
 		(property "Description" "Generic connectable mounting pin connector, single row, 01x03, script generated (kicad-library-utils/schlib/autogen/connector/)"
-			(at 54.61 210.82 0)
+			(at 54.61 195.58 0)
 			(effects
 				(font
@@
 		)
 		(property "LCSC" "C160403"
-			(at 54.61 210.82 0)
+			(at 54.61 195.58 0)
 			(effects
 				(font
@@
 			(project "control"
 				(path "/da26d94e-7a50-4b99-9678-5aaaf6987a15"
-					(reference "J4")
+					(reference "J2")
 					(unit 1)
 				)
@@
 	(symbol
 		(lib_id "Connector_Generic_MountingPin:Conn_01x03_MountingPin")
-		(at 54.61 195.58 0)
+		(at 54.61 210.82 0)
 		(mirror y)
 		(unit 1)
@@
 		(on_board yes)
 		(dnp no)
-		(property "Reference" "J2"
-			(at 52.07 194.6655 0)
+		(property "Reference" "J3"
+			(at 52.07 209.9055 0)
 			(effects
 				(font
@@
 		)
 		(property "Value" "SWD"
-			(at 52.07 197.2055 0)
+			(at 52.07 212.4455 0)
 			(effects
 				(font
@@
 		)
 		(property "Footprint" "Connector_JST:JST_SH_SM03B-SRSS-TB_1x03-1MP_P1.00mm_Horizontal"
-			(at 54.61 195.58 0)
+			(at 54.61 210.82 0)
 			(effects
 				(font
@@
 		)
 		(property "Datasheet" "~"
-			(at 54.61 195.58 0)
+			(at 54.61 210.82 0)
 			(effects
 				(font
@@
 		)
 		(property "Description" "Generic connectable mounting pin connector, single row, 01x03, script generated (kicad-library-utils/schlib/autogen/connector/)"
-			(at 54.61 195.58 0)
+			(at 54.61 210.82 0)
 			(effects
 				(font
@@
 		)
 		(property "LCSC" "C160403"
-			(at 54.61 195.58 0)
+			(at 54.61 210.82 0)
 			(effects
 				(font
@@
 			(project ""
 				(path "/da26d94e-7a50-4b99-9678-5aaaf6987a15"
-					(reference "J2")
+					(reference "J3")
 					(unit 1)
 				)
@@
 		(on_board yes)
 		(dnp no)
-		(property "Reference" "J3"
+		(property "Reference" "J4"
 			(at 90.17 190.5 0)
 			(effects
@@
 			(project "control"
 				(path "/da26d94e-7a50-4b99-9678-5aaaf6987a15"
-					(reference "J3")
+					(reference "J4")
 					(unit 1)
 				)
@@
 	(symbol
 		(lib_id "power:GND")
-		(at 62.23 215.9 0)
+		(at 62.23 200.66 0)
 		(unit 1)
 		(exclude_from_sim no)
@@
 		(fields_autoplaced yes)
 		(property "Reference" "#PWR0130"
-			(at 62.23 222.25 0)
+			(at 62.23 207.01 0)
 			(effects
 				(font
@@
 		)
 		(property "Value" "GND"
-			(at 62.23 220.98 0)
+			(at 62.23 205.74 0)
 			(effects
 				(font
@@
 		)
 		(property "Footprint" ""
-			(at 62.23 215.9 0)
+			(at 62.23 200.66 0)
 			(effects
 				(font
@@
 		)
 		(property "Datasheet" ""
-			(at 62.23 215.9 0)
+			(at 62.23 200.66 0)
 			(effects
 				(font
@@
 		)
 		(property "Description" "Power symbol creates a global label with name \"GND\" , ground"
-			(at 62.23 215.9 0)
+			(at 62.23 200.66 0)
 			(effects
 				(font
@@
 	(symbol
 		(lib_id "power:GND")
-		(at 62.23 200.66 0)
+		(at 62.23 215.9 0)
 		(unit 1)
 		(exclude_from_sim no)
@@
 		(fields_autoplaced yes)
 		(property "Reference" "#PWR0129"
-			(at 62.23 207.01 0)
+			(at 62.23 222.25 0)
 			(effects
 				(font
@@
 		)
 		(property "Value" "GND"
-			(at 62.23 205.74 0)
+			(at 62.23 220.98 0)
 			(effects
 				(font
@@
 		)
 		(property "Footprint" ""
-			(at 62.23 200.66 0)
+			(at 62.23 215.9 0)
 			(effects
 				(font
@@
 		)
 		(property "Datasheet" ""
-			(at 62.23 200.66 0)
+			(at 62.23 215.9 0)
 			(effects
 				(font
@@
 		)
 		(property "Description" "Power symbol creates a global label with name \"GND\" , ground"
-			(at 62.23 200.66 0)
+			(at 62.23 215.9 0)
 			(effects
 				(font

Commit message: Replace illuminated button with separate components
Parts:
- removed SW1: 228EMSARGFR, midi_concertina:CTS_228EMS, symbol midi_concertina:CTS_228E
- added D1: RED, LED_SMD:LED_0603_1608Metric, symbol Device:LED
- added D2, D3: ESD351, Diode_SMD:D_0402_1005Metric, symbol Device:D_Zener
- added LP1: ~, midi_concertina:SLP3-150-150-F, symbol midi_concertina:LightPipe
- added SW1: SYS, Button_Switch_SMD:Panasonic_EVQPUL_EVQPUC, symbol Switch:SW_Push
- H1: footprint MountingHole:MountingHole_3.2mm_M3 -> MountingHole:MountingHole_3.2mm_M3_Pad; symbol Mechanical:MountingHole -> Mechanical:MountingHole_Pad
Connections:
- net GND: now also H1.1, D1.1 (K), D2.2 (A), D3.2 (A), SW1.2
- net at U4.36 (GPIO24): now also D3.1 (K), SW1.1; no longer R8.1
- net at U4.37 (GPIO25): now also R8.1
- net at R8.2: now also D1.2 (A), D2.1 (K)
- no-connect marks 27 -> 28
Other:
- note added: "Mechanical"
- note removed: "Mounting Holes"
- moved on the sheet: C18, J5, R8, U5

Commit message: Update parts for controller board
Parts:
- C13, C14, C2, C3: LCSC C528974 -> C52923
- J1: LCSC C3020560 -> C2988369
- LP1: value ~ -> SLP-150-150-F; now in the parts list
Changed lines of the file:
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@@
 			)
 		)
-		(property "LCSC" "C528974"
+		(property "LCSC" "C52923"
 			(at 58.42 153.67 0)
 			(effects
@@
 			)
 		)
-		(property "Datasheet" "~"
+		(property "Datasheet" "https://www3.panasonic.biz/ac/cdn/e/control/switch/light-touch/catalog/sw_lt_eng_smalls_side.pdf"
 			(at 298.45 199.39 0)
 			(effects
@@
 			)
 		)
-		(property "Datasheet" "~"
+		(property "Datasheet" "https://mm.digikey.com/Volume0/opasdata/d220001/medias/docus/6536/ABM8_Datasheet.pdf"
 			(at 162.56 186.69 0)
 			(effects
@@
 			)
 		)
-		(property "LCSC" "C528974"
+		(property "LCSC" "C52923"
 			(at 353.06 76.2 0)
 			(effects
@@
 			)
 		)
-		(property "Datasheet" "~"
+		(property "Datasheet" "https://www.jst-mfg.com/product/pdf/eng/eSH.pdf"
 			(at 54.61 195.58 0)
 			(effects
@@
 			)
 		)
-		(property "Datasheet" "https://www.usb.org/sites/default/files/documents/usb_type-c.zip"
+		(property "Datasheet" "https://www.digikey.com/en/products/detail/gct/USB4105-GF-A/11198441"
 			(at 63.5 85.09 0)
 			(effects
@@
 			)
 		)
-		(property "LCSC" "C3020560"
+		(property "LCSC" "C2988369"
 			(at 59.69 85.09 0)
 			(effects
@@
 			)
 		)
-		(property "Datasheet" "~"
+		(property "Datasheet" "https://www.jst-mfg.com/product/pdf/eng/eSH.pdf"
 			(at 353.06 161.29 0)
 			(effects
@@
 			)
 		)
-		(property "Datasheet" "~"
+		(property "Datasheet" "https://www.jst-mfg.com/product/pdf/eng/eSH.pdf"
 			(at 54.61 210.82 0)
 			(effects
@@
 			)
 		)
-		(property "LCSC" "C528974"
+		(property "LCSC" "C52923"
 			(at 99.06 153.67 0)
 			(effects
@@
 			)
 		)
-		(property "LCSC" "C528974"
+		(property "LCSC" "C52923"
 			(at 304.8 76.2 0)
 			(effects
@@
 		(unit 1)
 		(exclude_from_sim no)
-		(in_bom no)
+		(in_bom yes)
 		(on_board yes)
 		(dnp no)
@@
 			)
 		)
-		(property "Value" "~"
+		(property "Value" "SLP-150-150-F"
 			(at 374.65 199.39 0)
 			(effects

Commit message: Replace I2C connector
Parts:
- added C19: 100n, Capacitor_SMD:C_0402_1005Metric, symbol Device:C
- added R6, R7: 2k2, Resistor_SMD:R_0402_1005Metric, symbol Device:R_US
- J5: value QWIIC -> I2C; footprint Connector_JST:JST_SH_SM04B-SRSS-TB_1x04-1MP_P1.00mm_Horizontal -> Connector_Molex:Molex_PicoBlade_53261-0471_1x04-1MP_P1.25mm_Horizontal; LCSC C160404 -> C5119769
- renumbered LP1 to H2, R9 to R10, R8 to R11, R10 to R12, R11 to R13, R6 to R4, R7 to R5, R4 to R8, R5 to R9
Connections:
- net +3.3V: now also C19.1, R6.1, R7.1
- net GND: now also J5.3 (Pin_3), C19.2; no longer J5.1 (Pin_1)
- net I2C_SCL: now also R7.2
- net I2C_SDA: now also J5.1 (Pin_1), R6.2; no longer J5.3 (Pin_3)
Other:
- note added: "Hardware"
- note removed: "Mechanical"
- moved on the sheet: H1, H2, J5
