File: electrical/Controller/Controller.kicad_pcb (KiCad board)
At the start: 2 copper layers, 72 x 20 mm, 30 parts, among them J1 USB4145-03-0170-C, J3 TC2030-NL, U1 LP5912-3.3DRV, U2 USBLC6-2P6, U3 STM32L072CBTx

Commit message: Minor corrections to controller design
Parts:
- C13, C3: value 100n -> 100nF
- D2: footprint Diode_SMD:D_0402_1005Metric -> Package_SON:Texas_DPY0002A_0.6x1mm_P0.65mm
- moved D2 0.15 mm to (130.9, 85.5)
Changed lines of the file:
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@@
 		(allow_soldermask_bridges_in_footprints no)
 		(tenting front back)
+		(aux_axis_origin 116 89)
 		(pcbplotparams
-			(layerselection 0x00000000_00000000_55555555_5755757f)
+			(layerselection 0x00000000_00000000_55555555_575575ff)
 			(plot_on_all_layers_selection 0x00000000_00000000_00000000_00000000)
 			(disableapertmacros no)
@@
 			)
 		)
-		(property "LCSC" "C99277"
+		(property "LCSC" "C17393620"
 			(at 0 0 90)
 			(unlocked yes)
@@
 			)
 		)
-		(property "Value" "100n"
+		(property "Value" "100nF"
 			(at 0 1.16 90)
 			(layer "F.Fab")
@@
 		)
 	)
-	(footprint "Diode_SMD:D_0402_1005Metric"
+	(footprint "Package_SON:Texas_DPY0002A_0.6x1mm_P0.65mm"
 		(layer "F.Cu")
-		(at 130.75 85.5 180)
-		(descr "Diode SMD 0402 (1005 Metric), square (rectangular) end terminal, IPC-7351 nominal, (Body size source: http://www.tortai-tech.com/upload/download/2011102023233369053.pdf), generated with kicad-footprint-generator")
-		(tags "diode")
+		(at 130.9 85.5 180)
+		(descr "X1SON 2 pin 0.6x1mm 0.375mm height package, https://www.ti.com/lit/ml/mpss034c/mpss034c.pdf, https://www.ti.com/lit/ds/symlink/tpd6e05u06.pdf")
+		(tags "X1SON")
 		(property "Reference" "D2"
 			(at 0 -1.25 0)
+			(unlocked yes)
 			(layer "F.SilkS")
 			(effects
@@
 		)
 		(property "Value" "ESD351"
-			(at 0 1.17 0)
+			(at 0 1.25 180)
+			(unlocked yes)
 			(layer "F.Fab")
-			(hide yes)
 			(effects
 				(font
@@
 		)
 		(property "Datasheet" "https://www.ti.com/lit/ds/symlink/esd351.pdf"
-			(at 0 0 0)
+			(at 0 0 180)
+			(unlocked yes)
 			(layer "F.Fab")
 			(hide yes)
@@
 		)
 		(property "Description" "30kV uni-directional TVS ESD protection diode, ROHS"
-			(at 0 0 0)
+			(at 0 0 180)
+			(unlocked yes)
 			(layer "F.Fab")
 			(hide yes)
@@
 		(attr smd)
 		(fp_circle
-			(center -1.09 0)
-			(end -1.04 0)
+			(center -0.8 0)
+			(end -0.69 0)
 			(stroke
 				(width 0.1)
 				(type solid)
 			)
-			(fill no)
+			(fill yes)
 			(layer "F.SilkS")
 		)
-		(fp_line
-			(start 0.93 0.47)
-			(end -0.93 0.47)
-			(stroke
-				(width 0.05)
-				(type solid)
-			)
-			(layer "F.CrtYd")
-		)
-		(fp_line
-			(start 0.93 -0.47)
-			(end 0.93 0.47)
-			(stroke
-				(width 0.05)
-				(type solid)
-			)
-			(layer "F.CrtYd")
-		)
-		(fp_line
-			(start -0.93 0.47)
-			(end -0.93 -0.47)
-			(stroke
-				(width 0.05)
-				(type solid)
-			)
-			(layer "F.CrtYd")
-		)
-		(fp_line
-			(start -0.93 -0.47)
-			(end 0.93 -0.47)
+		(fp_rect
+			(start -0.65 -0.45)
+			(end 0.65 0.45)
 			(stroke
 				(width 0.05)
 				(type solid)
 			)
+			(fill no)
 			(layer "F.CrtYd")
 		)
 		(fp_line
-			(start 0.5 0.25)
-			(end -0.5 0.25)
+			(start -0.2 0.3)
+			(end -0.2 -0.3)
 			(stroke
 				(width 0.1)
@@
 		)
 		(fp_line
-			(start 0.5 -0.25)
-			(end 0.5 0.25)
+			(start -0.3 0.3)
+			(end -0.3 -0.3)
 			(stroke
 				(width 0.1)
@@
 		)
 		(fp_line
-			(start -0.3 0.25)
-			(end -0.3 -0.25)
+			(start -0.4 0.3)
+			(end -0.4 -0.3)
 			(stroke
 				(width 0.1)
@@
 			(layer "F.Fab")
 		)
-		(fp_line
-			(start -0.4 0.25)
-			(end -0.4 -0.25)
-			(stroke
-				(width 0.1)
-				(type solid)
-			)
-			(layer "F.Fab")
-		)
-		(fp_line
-			(start -0.5 0.25)
-			(end -0.5 -0.25)
-			(stroke
-				(width 0.1)
-				(type solid)
-			)
-			(layer "F.Fab")
-		)
-		(fp_line
-			(start -0.5 -0.25)
-			(end 0.5 -0.25)
+		(fp_rect
+			(start -0.5 -0.3)
+			(end 0.5 0.3)
 			(stroke
 				(width 0.1)
 				(type solid)
 			)
+			(fill no)
 			(layer "F.Fab")
 		)
 		(fp_text user "${REFERENCE}"
-			(at 0 0 0)
+			(at 0 0 180)
 			(layer "F.Fab")
 			(effects
@@
 		)
 		(pad "1" smd roundrect
-			(at -0.485 0 180)
-			(size 0.59 0.64)
+			(at -0.35 0 180)
+			(size 0.3 0.5)
 			(layers "F.Cu" "F.Mask" "F.Paste")
 			(roundrect_rratio 0.25)
@@
 		)
 		(pad "2" smd roundrect
-			(at 0.485 0 180)
-			(size 0.59 0.64)
+			(at 0.35 0 180)
+			(size 0.3 0.5)
 			(layers "F.Cu" "F.Mask" "F.Paste")
 			(roundrect_rratio 0.25)
@@
 		)
 		(embedded_fonts no)
-		(model "${KICAD9_3DMODEL_DIR}/Diode_SMD.3dshapes/D_0402_1005Metric.wrl"
+		(model "${KICAD9_3DMODEL_DIR}/Package_SON.3dshapes/Texas_DPY0002A_0.6x1mm_P0.65mm.step"
 			(offset
 				(xyz 0 0 0)
@@
 			)
 		)
-		(property "Value" "100n"
+		(property "Value" "100nF"
 			(at 0 1.16 0)
 			(layer "F.Fab")
@@
 	)
 	(segment
+		(start 129.5 85.5)
+		(end 130.55 85.5)
+		(width 0.3)
+		(layer "F.Cu")
+		(net 2)
+	)
+	(segment
 		(start 177.75 76.48)
 		(end 176.75 76.48)
@@
 		(net 2)
 	)
-	(segment
-		(start 129.5 85.5)
-		(end 130.265 85.5)
-		(width 0.3)
-		(layer "F.Cu")
-		(net 2)
-	)
 	(via
 		(at 181.5 80.875)
@@
 	)
 	(segment
-		(start 132.5 87.75)
-		(end 131.235 86.485)
-		(width 0.15)
+		(start 131.25 83.55)
+		(end 131.25 85.5)
+		(width 0.3)
 		(layer "F.Cu")
 		(net 52)
 	)
 	(segment
-		(start 131.25 85.485)
-		(end 131.235 85.5)
-		(width 0.3)
+		(start 131.25 86.5)
+		(end 131.25 85.5)
+		(width 0.15)
 		(layer "F.Cu")
 		(net 52)
@@
 	)
 	(segment
-		(start 131.235 86.485)
-		(end 131.235 85.5)
+		(start 170.25 81.4125)
+		(end 170.25 85.25)
 		(width 0.15)
 		(layer "F.Cu")
@@
 	)
 	(segment
-		(start 170.25 81.4125)
-		(end 170.25 85.25)
+		(start 132.5 87.75)
+		(end 131.25 86.5)
 		(width 0.15)
 		(layer "F.Cu")
@@
 		(layer "F.Cu")
 		(net 52)
-	)
-	(segment
-		(start 131.25 83.55)
-		(end 131.25 85.485)
-		(width 0.3)
-		(layer "F.Cu")
-		(net 52)
