File: electrical/AngloLeftHand/AngloLeftHand.kicad_sch (KiCad schematic)
At the start: 49 parts, among them J3 TC2030-NL, U1 DRV5053VAQDBZR, U10 DRV5053VAQDBZR, U11 DRV5053VAQDBZR, U12 DRV5053VAQDBZR, U13 DRV5053VAQDBZR, U14 DRV5053VAQDBZR, U15 DRV5053VAQDBZR, U16 STM32L072CBTx, U17 CD74HC4067SM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

Commit message: Swap SDA and SCL on button board connectors
Connections:
- net I2C_SCL: now also J1.1 (Pin_1), J2.1 (Pin_1); no longer J1.3 (Pin_3), J2.3 (Pin_3)
- net I2C_SDA: now also J1.3 (Pin_3), J2.3 (Pin_3); no longer J1.1 (Pin_1), J2.1 (Pin_1)
Changed lines of the file:
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@@
 	(global_label "I2C_SDA"
 		(shape bidirectional)
-		(at 109.22 176.53 0)
-		(fields_autoplaced yes)
-		(effects
-			(font
-				(size 1.27 1.27)
-			)
-			(justify left)
-		)
-		(property "Intersheetrefs" "${INTERSHEET_REFS}"
-			(at 120.9365 176.53 0)
+		(at 109.22 181.61 0)
+		(fields_autoplaced yes)
+		(effects
+			(font
+				(size 1.27 1.27)
+			)
+			(justify left)
+		)
+		(property "Intersheetrefs" "${INTERSHEET_REFS}"
+			(at 120.9365 181.61 0)
 			(effects
 				(font
@@
 	(global_label "I2C_SCL"
 		(shape bidirectional)
-		(at 109.22 181.61 0)
-		(fields_autoplaced yes)
-		(effects
-			(font
-				(size 1.27 1.27)
-			)
-			(justify left)
-		)
-		(property "Intersheetrefs" "${INTERSHEET_REFS}"
-			(at 120.876 181.61 0)
+		(at 109.22 176.53 0)
+		(fields_autoplaced yes)
+		(effects
+			(font
+				(size 1.27 1.27)
+			)
+			(justify left)
+		)
+		(property "Intersheetrefs" "${INTERSHEET_REFS}"
+			(at 120.876 176.53 0)
 			(effects
 				(font
@@
 	(global_label "I2C_SDA"
 		(shape bidirectional)
-		(at 154.94 176.53 0)
-		(fields_autoplaced yes)
-		(effects
-			(font
-				(size 1.27 1.27)
-			)
-			(justify left)
-		)
-		(property "Intersheetrefs" "${INTERSHEET_REFS}"
-			(at 166.6565 176.53 0)
+		(at 154.94 181.61 0)
+		(fields_autoplaced yes)
+		(effects
+			(font
+				(size 1.27 1.27)
+			)
+			(justify left)
+		)
+		(property "Intersheetrefs" "${INTERSHEET_REFS}"
+			(at 166.6565 181.61 0)
 			(effects
 				(font
@@
 	(global_label "I2C_SCL"
 		(shape bidirectional)
-		(at 154.94 181.61 0)
-		(fields_autoplaced yes)
-		(effects
-			(font
-				(size 1.27 1.27)
-			)
-			(justify left)
-		)
-		(property "Intersheetrefs" "${INTERSHEET_REFS}"
-			(at 166.596 181.61 0)
-			(effects
-				(font
+		(at 154.94 176.53 0)
+		(fields_autoplaced yes)
+		(effects
+			(font
+				(size 1.27 1.27)
+			)
+			(justify left)
+		)
+		(property "Intersheetrefs" "${INTERSHEET_REFS}"
+			(at 166.596 176.53 0)
+			(effects
+				(font

Commit message: PCB adjustments
Parts:
- H1, H2: footprint MountingHole:MountingHole_3.2mm_M3_Pad -> MountingHole:MountingHole_3.2mm_M3; symbol Mechanical:MountingHole_Pad -> Mechanical:MountingHole
Connections:
- net GND: no longer H1.1, H2.1
Changed lines of the file:
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@@
 	(symbol
 		(lib_id "power:GND")
-		(at 116.84 232.41 0)
-		(unit 1)
-		(exclude_from_sim no)
-		(in_bom yes)
-		(on_board yes)
-		(dnp no)
-		(fields_autoplaced yes)
-		(property "Reference" "#PWR0118"
-			(at 116.84 238.76 0)
-			(effects
-				(font
-					(size 1.27 1.27)
-				)
-				(hide yes)
-			)
-		)
-		(property "Value" "GND"
-			(at 116.84 237.49 0)
-			(effects
-				(font
-					(size 1.27 1.27)
-				)
-				(hide yes)
-			)
-		)
-		(property "Footprint" ""
-			(at 116.84 232.41 0)
-			(effects
-				(font
-					(size 1.27 1.27)
-				)
-				(hide yes)
-			)
-		)
-		(property "Datasheet" ""
-			(at 116.84 232.41 0)
-			(effects
-				(font
-					(size 1.27 1.27)
-				)
-				(hide yes)
-			)
-		)
-		(property "Description" "Power symbol creates a global label with name \"GND\" , ground"
-			(at 116.84 232.41 0)
-			(effects
-				(font
-					(size 1.27 1.27)
-				)
-				(hide yes)
-			)
-		)
-		(pin "1"
-		)
-		(instances
-			(project "AngloRightHand"
-				(path "/da26d94e-7a50-4b99-9678-5aaaf6987a15"
-					(reference "#PWR0118")
-					(unit 1)
-				)
-			)
-		)
-	)
-	(symbol
-		(lib_id "power:GND")
 		(at 106.68 198.12 0)
 		(unit 1)
@@
 	)
 	(symbol
-		(lib_id "Mechanical:MountingHole_Pad")
+		(lib_id "Mechanical:MountingHole")
 		(at 96.52 229.87 0)
 		(unit 1)
@@
 			)
 		)
-		(property "Footprint" "MountingHole:MountingHole_3.2mm_M3_Pad"
+		(property "Footprint" "MountingHole:MountingHole_3.2mm_M3"
 			(at 96.52 229.87 0)
 			(effects
@@
 			)
 		)
-		(property "Description" "Mounting Hole with connection"
+		(property "Description" "Mounting Hole without connection"
 			(at 96.52 229.87 0)
 			(effects
@@
 			)
 		)
-		(pin "1"
-		)
 		(instances
 			(project "control"
@@
 	)
 	(symbol
-		(lib_id "power:GND")
-		(at 96.52 232.41 0)
-		(unit 1)
-		(exclude_from_sim no)
-		(in_bom yes)
-		(on_board yes)
-		(dnp no)
-		(fields_autoplaced yes)
-		(property "Reference" "#PWR0117"
-			(at 96.52 238.76 0)
-			(effects
-				(font
-					(size 1.27 1.27)
-				)
-				(hide yes)
-			)
-		)
-		(property "Value" "GND"
-			(at 96.52 237.49 0)
-			(effects
-				(font
-					(size 1.27 1.27)
-				)
-				(hide yes)
-			)
-		)
-		(property "Footprint" ""
-			(at 96.52 232.41 0)
-			(effects
-				(font
-					(size 1.27 1.27)
-				)
-				(hide yes)
-			)
-		)
-		(property "Datasheet" ""
-			(at 96.52 232.41 0)
-			(effects
-				(font
-					(size 1.27 1.27)
-				)
-				(hide yes)
-			)
-		)
-		(property "Description" "Power symbol creates a global label with name \"GND\" , ground"
-			(at 96.52 232.41 0)
-			(effects
-				(font
-					(size 1.27 1.27)
-				)
-				(hide yes)
-			)
-		)
-		(pin "1"
-		)
-		(instances
-			(project "control"
-				(path "/da26d94e-7a50-4b99-9678-5aaaf6987a15"
-					(reference "#PWR0117")
-					(unit 1)
-				)
-			)
-		)
-	)
-	(symbol
 		(lib_id "MidiConcertina:TI_DRV5053xDBZ")
 		(at 340.36 125.73 0)
@@
 	)
 	(symbol
-		(lib_id "Mechanical:MountingHole_Pad")
+		(lib_id "Mechanical:MountingHole")
 		(at 116.84 229.87 0)
 		(unit 1)
@@
 			)
 		)
-		(property "Footprint" "MountingHole:MountingHole_3.2mm_M3_Pad"
+		(property "Footprint" "MountingHole:MountingHole_3.2mm_M3"
 			(at 116.84 229.87 0)
 			(effects
@@
 			)
 		)
-		(property "Description" "Mounting Hole with connection"
+		(property "Description" "Mounting Hole without connection"
 			(at 116.84 229.87 0)
 			(effects
@@
 			)
 		)
-		(pin "1"
-		)
 		(instances

Commit message: Add licenses
Other:
- company: Bushel Basket Musical Instruments -> (none)
Changed lines of the file:
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@@
 	(title_block
 		(title "MIDI Concertina Controller")
-		(company "Bushel Basket Musical Instruments")
+		(comment 1 "https://ohwr.org/cern_ohl_s_v2.pdf")
+		(comment 2 "Licensed under CERN-OHL-S v2 or any later version")
+		(comment 3 "Copyright 2025 Steven Schulteis")
 	)
 	(junction

Commit message: Minor corrections to left hand board
Parts:
- C1, C10, C11, C12, C13, C14, C15, C2, C22, C24, C25, C3, C4, C5, C6, C7, C8, C9: value 100n -> 100nF
- J1, J2: LCSC C99277 -> C17393620
