File: electrical/AngloRightHand/AngloRightHand.kicad_pcb (KiCad board)
At the start: 2 copper layers, 82 x 60 mm, 47 parts, among them J1 I2C, J2 TC2030-NL, U1 DRV5053VAQDBZR, U10 DRV5053VAQDBZR, U11 DRV5053VAQDBZR, U12 DRV5053VAQDBZR, U13 DRV5053VAQDBZR, U14 DRV5053VAQDBZR, U15 DRV5053VAQDBZR, U16 STM32L072CBTx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

Commit message: Use TITLE variable in silkscreen
Other:
- board text added: "${TITLE} - Rev ${REVISION}"
- board text removed: "MIDI Anglo Right Hand - Rev ${REVISION}"
Changed lines of the file:
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@@
 		(layer "Edge.Cuts")
 	)
-	(gr_text "MIDI Anglo Right Hand - Rev ${REVISION}"
+	(gr_text "${TITLE} - Rev ${REVISION}"
 		(at 80 106 0)
 		(layer "B.SilkS")
