File: electrical/AngloRightKeyboard/AngloRightKeyboard.kicad_pcb (KiCad board)
At the start: 2 copper layers, 82 x 60 mm, 47 parts, among them J1 I2C, J2 TC2030-NL, U1 DRV5053VAQDBZR, U10 DRV5053VAQDBZR, U11 DRV5053VAQDBZR, U12 DRV5053VAQDBZR, U13 DRV5053VAQDBZR, U14 DRV5053VAQDBZR, U15 DRV5053VAQDBZR, U16 STM32L072CBTx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

Commit message: Change i2c cable pinout to keep signals between grounds
Parts:
- moved C24 5.75 mm to (69.2, 160.7), turned to -90 degrees
Connections:
- J1 pad 1: I2C_SCL -> GND
- J1 pad 2: GND -> I2C_SCL
- J1 pad 3: I2C_SDA -> GND
- J1 pad 4: GND -> I2C_SDA
- J1 pad 5: +3.3V -> GND
- J1 pad 6: GND -> +3.3V
Routing:
- net +3.3V: track 122.2 -> 115.7 mm
- net I2C_SDA: track 31.0 -> 29.7 mm
- net I2C_SCL: track 33.3 -> 32.1 mm
- net GND: vias 496 -> 498
