File: electrical/AngloRightKeyboard/AngloRightKeyboard.kicad_sch (KiCad schematic)
At the start: 47 parts, among them J1 I2C, J2 TC2030-NL, U1 DRV5053VAQDBZR, U10 DRV5053VAQDBZR, U11 DRV5053VAQDBZR, U12 DRV5053VAQDBZR, U13 DRV5053VAQDBZR, U14 DRV5053VAQDBZR, U15 DRV5053VAQDBZR, U16 STM32L072CBTx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

Commit message: Exclude I2C connectors from BOM
Parts:
- J1: now left out of the parts list
Changed lines of the file:
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@@
 		(unit 1)
 		(exclude_from_sim no)
-		(in_bom yes)
+		(in_bom no)
 		(on_board yes)
 		(dnp no)
