File: electrical/BellowsSensor/BellowsSensor.kicad_sch (KiCad schematic)
At the start: 5 parts, among them J1 I2C, U1 ELVH-001D-HRRJ-C-N2A4

Commit message: Exclude I2C connectors from BOM
Parts:
- J1: now left out of the parts list
Changed lines of the file:
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@@
 		(unit 1)
 		(exclude_from_sim no)
-		(in_bom yes)
+		(in_bom no)
 		(on_board yes)
 		(dnp no)
