File: electrical/BellowsSensorA/BellowsSensorA.kicad_sch (KiCad schematic)
At the start: 5 parts, among them J1 I2C, U1 ELVH-001D-HRRJ-C-N2A4

Commit message: Switch pressure sensor for BellowsSensorA
Parts:
- removed U1: ELVH-001D-HRRJ-C-N2A4, MidiConcertina:Amphenol_ELVH-x-xJ-x-x, symbol MidiConcertina:Amphenol_ELVH-x
- added U1: CPS610DSD010DH01, Package_SO:SOIC-16W_7.5x10.3mm_P1.27mm, symbol MidiConcertina:Consensic_CPS610x
Connections:
- net +3.3V: now also U1.7 (VDD)
- net GND: now also U1.6 (GND)
- net I2C_SCL: now also U1.11 (SCL)
- net I2C_SDA: now also U1.10 (SDA)
Changed lines of the file:
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@@
-	)
-	(symbol
-		(lib_id "MidiConcertina:Amphenol_ELVH-x")
-		(at 158.75 80.01 0)
-		(mirror y)
-		(unit 1)
-		(exclude_from_sim no)
-		(in_bom yes)
-		(on_board yes)
-		(dnp no)
-		(property "Reference" "U1"
-			(at 156.21 67.31 0)
-			(effects
-				(font
-					(size 1.27 1.27)
-				)
-				(justify left)
-			)
-		)
-		(property "Value" "ELVH-001D-HRRJ-C-N2A4"
-			(at 156.21 69.85 0)
-			(effects
-				(font
-					(size 1.27 1.27)
-				)
-				(justify left)
-			)
-		)
-		(property "Footprint" "MidiConcertina:Amphenol_ELVH-x-xJ-x-x"
-			(at 158.75 80.01 0)
-			(effects
-				(font
-					(size 1.27 1.27)
-				)
-				(hide yes)
-			)
-		)
-		(property "Datasheet" "https://428059.fs1.hubspotusercontent-na1.net/hubfs/428059/Product-Data-Sheets/DS-0376.pdf"
-			(at 158.75 80.01 0)
-			(effects
-				(font
-					(size 1.27 1.27)
-				)
-				(hide yes)
-			)
-		)
-		(property "Description" "Pressure Sensor ±1PSI (±6.89kPa) Differential Male - 0.06\" (1.6mm) Tube, Dual Ports, Same Side, ROHS"
-			(at 158.75 80.01 0)
-			(effects
-				(font
-					(size 1.27 1.27)
-				)
-				(hide yes)
-			)
-		)
-		(property "LCSC" "C3241336"
-			(at 158.75 80.01 0)
-			(effects
-				(font
-					(size 1.27 1.27)
-				)
-				(hide yes)
-			)
-		)
-		(property "Part" "Amphenol ELVH-001D-HRRJ-C-N2A4"
-			(at 158.75 80.01 0)
-			(effects
-				(font
-					(size 1.27 1.27)
-				)
-				(hide yes)
-			)
-		)
-		(pin "8"
-		)
-		(pin "4"
-		)
-		(pin "1"
-		)
-		(pin "3"
-		)
-		(pin "6"
-		)
-		(pin "7"
-		)
-		(pin "2"
-		)
-		(pin "5"
-		)
-		(instances
-			(project ""
-				(path "/ceae7089-9cb4-4950-bb64-2f75302207fd"
-					(reference "U1")
-					(unit 1)
-				)
-			)
-		)
 	)
 	(symbol
@@
 					(unit 1)
 				)
+			)
+		)
+	)
+	(symbol
+		(lib_id "MidiConcertina:Consensic_CPS610x")
+		(at 158.75 80.01 0)
+		(mirror y)
+		(unit 1)
+		(exclude_from_sim no)
+		(in_bom yes)
+		(on_board yes)
+		(dnp no)
+		(property "Reference" "U1"
+			(at 156.21 67.31 0)
+			(effects
+				(font
+					(size 1.27 1.27)
+				)
+				(justify left)
+			)
+		)
+		(property "Value" "CPS610DSD010DH01"
+			(at 156.21 69.85 0)
+			(effects
+				(font
+					(size 1.27 1.27)
+				)
+				(justify left)
+			)
+		)
+		(property "Footprint" "Package_SO:SOIC-16W_7.5x10.3mm_P1.27mm"
+			(at 158.75 80.01 0)
+			(effects
+				(font
+					(size 1.27 1.27)
+				)
+				(hide yes)
+			)
+		)
+		(property "Datasheet" "https://jlcpcb.com/api/file/downloadByFileSystemAccessId/8603406260650205184"
+			(at 158.75 80.01 0)
+			(effects
+				(font
+					(size 1.27 1.27)
+				)
+				(hide yes)
+			)
+		)
+		(property "Description" "Pressure Sensor ±10kPa Differential Male - 2.2mm Tube, Dual Ports, ROHS"
+			(at 158.75 80.01 0)
+			(effects
+				(font
+					(size 1.27 1.27)
+				)
+				(hide yes)
+			)
+		)
+		(property "LCSC" "C28646450"
+			(at 158.75 80.01 0)
+			(effects
+				(font
+					(size 1.27 1.27)
+				)
+				(hide yes)
+			)
+		)
+		(property "Part" "Consensic CPS610DSD010DH01"
+			(at 158.75 80.01 0)
+			(effects
+				(font
+					(size 1.27 1.27)
+				)
+				(hide yes)
+			)
+		)
+		(pin "14"
+		)
+		(pin "15"
+		)
+		(pin "16"
+		)
+		(pin "2"
+		)
+		(pin "3"
+		)
+		(pin "4"
+		)
+		(pin "5"
+		)
+		(pin "8"
+		)
+		(pin "9"
+		)
+		(pin "7"
+		)
+		(pin "12"
+		)
+		(pin "13"
+		)
+		(pin "6"
+		)
+		(pin "11"
+		)
+		(pin "10"
+		)
+		(pin "1"
+		)
+		(instances
+			(project ""
+				(path "/ceae7089-9cb4-4950-bb64-2f75302207fd"
+					(reference "U1")
+					(unit 1)
+				)

Commit message: Update bellows sensor labels
Other:
- title: MIDI Bellows Sensor -> MIDI Bellows Sensor A
Changed lines of the file:
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@@
 	(paper "USLetter")
 	(title_block
-		(title "MIDI Bellows Sensor")
+		(title "MIDI Bellows Sensor A")
 		(date "2026-01-19")
 		(rev "1")
